File: hardware/pcb/opencalc_pcb_V5/opencalc_pcb_V5.kicad_pcb (KiCad board)
At the start: 4 copper layers, 75 x 170 mm, 180 parts, among them J1 FH12-18S-0.5SH55, J3 USB4085-GF-A, Q1 AO3401A, SW1 RESET, SW10 Button8, SW11 Button9, SW12 Button10, SW13 Button11, SW14 Button12, SW15 Button13, SW16 Button14, SW17 Button15, SW18 Button16, SW19 Button17, SW2 BOOT, SW20 Button18, SW21 Button19, SW22 Button20, SW23 Button21, SW24 Button22, SW25 Button23, SW26 Button24, SW27 Button25, SW28 Button26, SW29 Button27, SW3 Button1, SW30 Button28, SW31 Button29, SW32 Button30, SW33 Button31, SW34 Button32, SW35 Button33, SW36 Button34, SW37 Button35, SW38 Button36, SW39 Button37, SW4 Button2, SW40 Button38, SW41 Button39, SW42 Button40, SW43 Button41, SW44 Button42, SW45 Button43, SW46 Button44, SW47 Button45, SW48 Button46, SW49 Button47, SW5 Button3, SW50 Button48, SW51 Button49, SW52 Button50, SW53 SW_SPDT, SW6 Button4, SW7 Button5, SW8 Button6, SW9 Button7, U1 ESP32-S3-WROOM-1-N16R8, U2 TPS63802DLAR, U3 TPD2E2U06DCKR, U4 BQ24074RGTR, U5 PAM8302AADCR, U6 CMS-151504-SMT-TR

Commit message: Update OpenCalc
Other:
- board text added: "Made By Cory Pearl"
Changed lines of the file:
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@@
+		)
+	)
+	(gr_text "Made By Cory Pearl"
+		(at 68.1 71.1 0)
+		(layer "B.SilkS")
+		(effects
+			(font
+				(size 1.5 1.5)
+				(thickness 0.3)
+				(bold yes)
+			)
+			(justify left bottom mirror)
 		)
 	)

Commit message: big software, readme, and blog
Parts:
- added C18: 100nF, Capacitor_SMD:C_0805_2012Metric_Pad1.18x1.45mm_HandSolder, B.Cu at (25.0, 27.3)
- added C19: 100nF, Capacitor_SMD:C_0805_2012Metric_Pad1.18x1.45mm_HandSolder, B.Cu at (40.2, 40.7)
- added J2: PPTC152LFBN-RC, opencalc_footprint_library:PPTC152LFBN_RC, B.Cu at (63.0, 21.5)
- added R35: 10kΩ, Resistor_SMD:R_0805_2012Metric_Pad1.20x1.40mm_HandSolder, B.Cu at (31.9, 32.1)
- added R36: 10kΩ, Resistor_SMD:R_0805_2012Metric_Pad1.20x1.40mm_HandSolder, B.Cu at (30.6, 38.8)
- added R37: 10kΩ, Resistor_SMD:R_0805_2012Metric_Pad1.20x1.40mm_HandSolder, B.Cu at (23.6, 38.1)
- added R38: 4.7kΩ, Resistor_SMD:R_0805_2012Metric_Pad1.20x1.40mm_HandSolder, B.Cu at (54.4, 38.4)
- added R39: 4.7kΩ, Resistor_SMD:R_0805_2012Metric_Pad1.20x1.40mm_HandSolder, B.Cu at (53.0, 29.8)
- added U7: ADS1115IDGST, opencalc_footprint_library:ADS1115IDGST, B.Cu at (26.5, 32.5)
- added U8: MCP23017T-E/SO, opencalc_footprint_library:MCP23017T_E_SO, B.Cu at (42.4, 33.7)
- C1, C10, C11, C12, C13, C14, C15, C16, C17, C2, C3, C4, C5, C6, C7, C8, C9: footprint Capacitor_SMD:C_0603_1608Metric -> Capacitor_SMD:C_0805_2012Metric_Pad1.18x1.45mm_HandSolder
- D1, D2, D3: footprint LED_SMD:LED_0603_1608Metric -> LED_SMD:LED_0805_2012Metric_Pad1.15x1.40mm_HandSolder
- D10, D11, D12, D13, D14, D15, D16, D17, D18, D19, D20, D21, D22, D23, D24, D25, D26, D27, D28, D29, D30, D31, D32, D33, D34, D35, D36, D37, D38, D39, D4, D40, D41, D42, D43, D44, D45, D46, D47, D48, D49, D5, D50, D51, D52, D53, D6, D7, D8, D9: footprint Diode_SMD:D_SOD-523 -> Diode_SMD:D_0805_2012Metric_Pad1.15x1.40mm_HandSolder
- R1, R10, R11, R12, R13, R14, R15, R17, R18, R19, R2, R20, R21, R22, R23, R24, R25, R26, R27, R28, R29, R3, R30, R31, R32, R33, R34, R4, R5, R6, R7, R8, R9: footprint Resistor_SMD:R_0603_1608Metric -> Resistor_SMD:R_0805_2012Metric_Pad1.20x1.40mm_HandSolder
- R16: value 4.4kΩ -> 2kΩ; footprint Resistor_SMD:R_0603_1608Metric -> Resistor_SMD:R_0805_2012Metric_Pad1.20x1.40mm_HandSolder
- moved R1 25.6 mm to (87.1, 21.2)
- moved D1 24.7 mm to (82.1, 21.2)
- moved C7 4.66 mm to (68.0, 62.6), turned to 90 degrees
- moved SW1 4.61 mm to (75.2, 62.7)
- moved TP4 4.51 mm to (78.9, 56.7)
- moved R3 3.67 mm to (83.9, 23.5)
- moved D44 3.64 mm to (35.4, 169.9)
- moved D23 3.26 mm to (83.6, 119.0)
- moved D4 2.72 mm to (36.0, 87.0)
- moved TP3 2.65 mm to (48.5, 173.4)
- moved R18 2.30 mm to (27.4, 141.9)
- moved D40 2.18 mm to (48.9, 159.4)
- moved D39 2.04 mm to (36.6, 159.0)
- moved C8 1.94 mm to (38.1, 87.1), turned to -90 degrees
- moved D25 1.84 mm to (49.0, 129.1)
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Connections:
- R2 pad 1: GND -> +3V3
- R3 pad 2: GND -> +3V3
- U1 pad 21: /AUDIO_SD -> /SDA
- U1 pad 23: /PWR_LED -> /SCL
Routing:
- net /SDA: track 0.00 -> 67.7 mm, vias 0 -> 2
- net /SCL: track 0.00 -> 59.4 mm, vias 0 -> 2
- net /COL0: track 170.5 -> 205.7 mm, vias 22 -> 16
- net /PWR_LED: track 21.7 -> 52.0 mm, vias 3 -> 1
- net +3V3: track 73.6 -> 103.2 mm, vias 20 -> 28
- net /DPIN0: track 0.00 -> 25.8 mm
- net /DPIN6: track 0.00 -> 25.7 mm, vias 0 -> 2
- net /APIN0: track 0.00 -> 25.4 mm, vias 0 -> 1
- net /DPIN8: track 0.00 -> 24.9 mm, vias 0 -> 2
- net /APIN1: track 0.00 -> 24.8 mm, vias 0 -> 1
- net /DPIN1: track 0.00 -> 24.8 mm, vias 0 -> 2
- net /DPIN7: track 0.00 -> 24.7 mm, vias 0 -> 2
- net GND: track 140.5 -> 164.3 mm, vias 39 -> 43
- net /COL1: track 139.5 -> 162.4 mm, vias 21 -> 14
- net /ADS_RDY: track 0.00 -> 22.5 mm, vias 0 -> 2
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Other:
- board text added: "+ HERE PLS ->"
- board text added: "."
- board text added: "1 3 5 7 9 11 13 15 17 19 21 23 25 27 29 2 4 6 8 10 12 14 16 18 20 22 24 26 28 30"

Commit message: removed files
Parts:
- R34: value 10k -> DNP
- R36: value 10kΩ -> 100kΩ
- moved F1 2.77 mm to (58.0, 179.0)
Connections:
- C10 pad 1: Net-(C10-Pad1) -> GND
- C11 pad 2: Net-(C10-Pad1) -> /USB_VBUS
Routing:
- net /USB_VBUS: track 23.7 -> 33.3 mm
- net GND: track 164.3 -> 168.3 mm
- net /AUDIO_SD: track 66.5 -> 70.4 mm
- net /VBUS_FUSE: track 16.6 -> 13.7 mm
- net Net-(C10-Pad1): track 2.66 -> 0.00 mm
Changed lines of the file:
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@@
 	(net 3 "/RESET_PIN")
 	(net 4 "/VBAT")
-	(net 5 "Net-(C10-Pad1)")
 	(net 6 "/USB_VBUS")
 	(net 7 "/VBAT_DIV")
@@
 			(layers "B.Cu" "B.Mask" "B.Paste")
 			(roundrect_rratio 0.212766)
-			(net 5 "Net-(C10-Pad1)")
+			(net 2 "GND")
 			(pintype "passive")
 		)
@@
 			)
 		)
-		(property "Value" "10k"
+		(property "Value" "DNP"
 			(at 0 -1.65 0)
 			(layer "B.Fab")
@@
 		(sheetname "/")
 		(sheetfile "opencalc_pcb_V5.kicad_sch")
-		(attr smd)
+		(attr smd dnp)
 		(fp_line
 			(start -0.227064 0.735)
@@
 	(footprint "Fuse:Fuse_1206_3216Metric"
 		(layer "B.Cu")
-		(at 58 176.2 180)
+		(at 58.02 178.97 180)
 		(descr "Fuse SMD 1206 (3216 Metric), square (rectangular) end terminal, IPC-7351 nominal, (Body size source: http://www.tortai-tech.com/upload/download/2011102023233369053.pdf), generated with kicad-footprint-generator")
 		(tags "fuse")
@@
 		)
 		(fp_line
-			(start -0.000003 -0.499999)
-			(end -0.000003 0.500002)
-			(stroke
-				(width 0.1)
-				(type solid)
-			)
-			(layer "B.CrtYd")
-		)
-		(fp_line
-			(start -0.500002 0)
-			(end 0.499999 0)
-			(stroke
-				(width 0.1)
-				(type solid)
-			)
-			(layer "B.CrtYd")
-		)
-		(fp_line
 			(start -3.150001 1.800001)
 			(end 3.149999 1.800001)
@@
 			(layers "B.Cu" "B.Mask" "B.Paste")
 			(roundrect_rratio 0.212766)
-			(net 5 "Net-(C10-Pad1)")
+			(net 6 "/USB_VBUS")
 			(pintype "passive")
 		)
@@
 			)
 		)
-		(property "Value" "10kΩ"
+		(property "Value" "100kΩ"
 			(at 0 -1.65 0)
 			(layer "B.Fab")
@@
 	(gr_line
 		(start 95 25)
-		(end 95 185)
+		(end 95 32.8)
 		(stroke
 			(width 0.05)
@@
 		(layer "Edge.Cuts")
 	)
-	(gr_rect
+	(gr_line
+		(start 95 32.8)
+		(end 88.2 32.8)
+		(stroke
+			(width 0.05)
+			(type default)
+		)
+		(layer "Edge.Cuts")
+	)
+	(gr_line
 		(start 88.2 32.8)
+		(end 88.2 51.4)
+		(stroke
+			(width 0.05)
+			(type default)
+		)
+		(layer "Edge.Cuts")
+	)
+	(gr_line
+		(start 88.2 51.4)
 		(end 95 51.4)
 		(stroke
 			(width 0.05)
-			(type dash)
+			(type default)
+		)
+		(layer "Edge.Cuts")
+	)
+	(gr_line
+		(start 95 51.4)
+		(end 95 185)
+		(stroke
+			(width 0.05)
+			(type default)
 		)
-		(fill no)
 		(layer "Edge.Cuts")
 	)
@@
 	)
 	(segment
+		(start 38.65 176.05)
+		(end 40.0625 177.4625)
+		(width 0.2)
+		(layer "B.Cu")
+		(net 2)
+	)
+	(segment
+		(start 40.0625 177.4625)
+		(end 42 177.4625)
+		(width 0.2)
+		(layer "B.Cu")
+		(net 2)
+	)
+	(segment
 		(start 89.825 65.86)
 		(end 91.46 65.86)
@@
 	)
 	(segment
-		(start 42 177.2)
-		(end 42 179.8625)
+		(start 42 179.8625)
+		(end 44 181.8625)
 		(width 0.75)
 		(layer "B.Cu")
-		(net 5)
+		(net 6)
 	)
 	(segment
-		(start 51.6 176.2)
-		(end 46.1 176.2)
+		(start 44 181.8625)
+		(end 44 176.2)
 		(width 0.75)
 		(layer "B.Cu")
@@
 	)
 	(segment
+		(start 56.62 178.97)
+		(end 53.85 176.2)
+		(width 0.75)
+		(layer "B.Cu")
+		(net 6)
+	)
+	(segment
 		(start 46.1 175.9)
 		(end 48.55 173.45)
@@
 	)
 	(segment
-		(start 56.6 176.2)
-		(end 51.6 176.2)
+		(start 53.85 176.2)
+		(end 46.1 176.2)
 		(width 0.75)
 		(layer "B.Cu")
@@
 	)
 	(segment
-		(start 59.6 184.35)
-		(end 59.6 183)
-		(width 0.2)
-		(layer "B.Cu")
-		(net 67)
-	)
-	(segment
-		(start 55.350001 184.25)
-		(end 55.350001 185.6)
+		(start 59.42 183.9)
+		(end 59.42 178.97)
 		(width 0.2)
 		(layer "B.Cu")
@@
 	)
 	(segment
-		(start 55.350001 184.35)
-		(end 55.350001 184.449999)
+		(start 59.6 184.25)
+		(end 59.6 184.08)
 		(width 0.2)
 		(layer "B.Cu")
@@
 	)
 	(segment
-		(start 59.6 181.25)
-		(end 59.6 178.2)
+		(start 55.350001 184.25)
+		(end 55.350001 185.6)
 		(width 0.2)
 		(layer "B.Cu")
@@
 	)
 	(segment
-		(start 59.6 183)
-		(end 59.7 182.9)
+		(start 55.350001 184.35)
+		(end 55.350001 184.449999)
 		(width 0.2)
 		(layer "B.Cu")
@@
 	)
 	(segment
-		(start 59.7 182.9)
-		(end 59.7 181.35)
+		(start 59.6 184.08)
+		(end 59.42 183.9)
 		(width 0.2)
 		(layer "B.Cu")
@@
 	)
 	(segment
-		(start 59.6 178.2)
-		(end 59.4 178)
-		(width 0.2)
-		(layer "B.Cu")
-		(net 67)
-	)
-	(segment
-		(start 59.7 181.35)
-		(end 59.6 181.25)
-		(width 0.2)
-		(layer "B.Cu")
-		(net 67)
-	)
-	(segment
-		(start 59.4 178)
-		(end 59.4 176.2)
-		(width 0.2)
-		(layer "B.Cu")
-		(net 67)
-	)
-	(segment
 		(start 72.4 43.2)
 		(end 78.2 49)
@@
 		(width 0.2)
 		(layer "B.Cu")
+		(net 126)
+	)
+	(segment
+		(start 46.575 82.7)
+		(end 46.575 86.63)
+		(width 0.2)
+		(layer "B.Cu")

Commit message: website added
Parts:
- added C20: 10nF, Capacitor_SMD:C_0805_2012Metric_Pad1.18x1.45mm_HandSolder, B.Cu at (47.7, 76.6)
- added C21: 10nF, Capacitor_SMD:C_0805_2012Metric_Pad1.18x1.45mm_HandSolder, B.Cu at (47.5, 71.0)
- added R40: 1kΩ, Resistor_SMD:R_0805_2012Metric_Pad1.20x1.40mm_HandSolder, B.Cu at (50.9, 70.0)
- added R41: 1kΩ, Resistor_SMD:R_0805_2012Metric_Pad1.20x1.40mm_HandSolder, B.Cu at (50.9, 75.5)
- R33: value 33Ω -> 1Ω
Connections:
- C16 pad 1: /AUDIO_OUT -> Net-(C16-Pad1)
Routing:
- net /AUDIO_OUT: track 70.1 -> 50.7 mm
- net /ROW1: track 128.9 -> 145.1 mm
- net Net-(C16-Pad1): track 0.00 -> 13.5 mm
- net GND: track 168.3 -> 156.5 mm, vias 43 -> 50
- net Net-(C21-Pad1): track 0.00 -> 5.88 mm
