File: hardware/pcb/opencalc_pcb_V5/opencalc_pcb_V5.kicad_sch (KiCad schematic)
At the start: 1 part, among them U1 ESP32-S3-WROOM-1-N16R8

Commit message: readme and sound update
Parts:
- removed U1: ESP32-S3-WROOM-1-N16R8, ESP32-S3-WROOM-1-N16R8, symbol opencalc:ESP32-S3-WROOM-1-N16R8
- added C1, C7, C8: 1uF, Capacitor_SMD:C_0603_1608Metric, symbol Device:C
- added C10, C12, C16, C17, C3, C4, C5, C6: 100nF, Capacitor_SMD:C_0603_1608Metric, symbol Device:C
- added C11: 4.7uF, Capacitor_SMD:C_0603_1608Metric, symbol Device:C
- added C13, C15, C2, C9: 10uF, Capacitor_SMD:C_0603_1608Metric, symbol Device:C
- added C14: 22uF, Capacitor_SMD:C_0603_1608Metric, symbol Device:C
- added D1: RED, LED_SMD:LED_0603_1608Metric, symbol Device:LED
- added D10, D11, D12, D13, D14, D15, D16, D17, D18, D19, D20, D21, D22, D23, D24, D25, D26, D27, D28, D29, D30, D31, D32, D33, D34, D35, D36, D37, D38, D39, D4, D40, D41, D42, D43, D44, D45, D46, D47, D48, D49, D5, D50, D51, D52, D53, D6, D7, D8, D9: 1N4148WT, Diode_SMD:D_SOD-523, symbol Diode:1N4148WT
- added D2: BLUE, LED_SMD:LED_0603_1608Metric, symbol Device:LED
- added D3: GREEN, LED_SMD:LED_0603_1608Metric, symbol Device:LED
- added F1: MF-NSMF200-2, Fuse:Fuse_1206_3216Metric, symbol Device:Polyfuse
- added J1: FH12-18S-0.5SH55, opencalc_footprint_library:FH12-18S-0.5SH(55), symbol opencalc_library:FH12-18S-0.5SH55
- added J3: USB4085-GF-A, opencalc_footprint_library:USB4085-GF-A, symbol opencalc_library:USB4085-GF-A
- added L1: 74479275147, opencalc_footprint_library:74479275147, symbol opencalc_library:74479275147
- added Q1: AO3401A, Package_TO_SOT_SMD:SOT-23, symbol Transistor_FET:AO3401A
- added R1, R12, R13: 1kΩ, Resistor_SMD:R_0603_1608Metric, symbol Device:R
- added R10, R9: 5.1kΩ, Resistor_SMD:R_0603_1608Metric, symbol Device:R
- added R11, R2, R3: 10kΩ, Resistor_SMD:R_0603_1608Metric, symbol Device:R
- added R14: 590Ω, Resistor_SMD:R_0603_1608Metric, symbol Device:R
- added R15: 1.1kΩ, Resistor_SMD:R_0603_1608Metric, symbol Device:R
- added R16: 4.4kΩ, Resistor_SMD:R_0603_1608Metric, symbol Device:R
- added R17: 46.4kΩ, Resistor_SMD:R_0603_1608Metric, symbol Device:R
- added R18, R19: 1MΩ, Resistor_SMD:R_0603_1608Metric, symbol Device:R
- added R20: 560kΩ, Resistor_SMD:R_0603_1608Metric, symbol Device:R
- added R21, R8: 100kΩ, Resistor_SMD:R_0603_1608Metric, symbol Device:R
- added R22, R23, R24, R25, R26, R27, R28, R29, R30, R31: 46kΩ, Resistor_SMD:R_0603_1608Metric, symbol Device:R
- added R32: 100Ω, Resistor_SMD:R_0603_1608Metric, symbol Device:R
- added R33: 33Ω, Resistor_SMD:R_0603_1608Metric, symbol Device:R
- added R34: 10k, Resistor_SMD:R_0603_1608Metric, symbol Device:R
- added R4, R5, R6, R7: 27Ω, Resistor_SMD:R_0603_1608Metric, symbol Device:R
- added SW1: RESET, Button_Switch_SMD:SW_Push_1P1T_NO_E-Switch_TL3301NxxxxxG, symbol Switch:SW_Push
- added SW10: Button8, Button_Switch_SMD:SW_Push_1P1T_NO_E-Switch_TL3301NxxxxxG, symbol Switch:SW_Push
- added SW11: Button9, Button_Switch_SMD:SW_Push_1P1T_NO_E-Switch_TL3301NxxxxxG, symbol Switch:SW_Push
- added SW12: Button10, Button_Switch_SMD:SW_Push_1P1T_NO_E-Switch_TL3301NxxxxxG, symbol Switch:SW_Push
- added SW13: Button11, Button_Switch_SMD:SW_Push_1P1T_NO_E-Switch_TL3301NxxxxxG, symbol Switch:SW_Push
- added SW14: Button12, Button_Switch_SMD:SW_Push_1P1T_NO_E-Switch_TL3301NxxxxxG, symbol Switch:SW_Push
- added SW15: Button13, Button_Switch_SMD:SW_Push_1P1T_NO_E-Switch_TL3301NxxxxxG, symbol Switch:SW_Push
- added SW16: Button14, Button_Switch_SMD:SW_Push_1P1T_NO_E-Switch_TL3301NxxxxxG, symbol Switch:SW_Push
- added SW17: Button15, Button_Switch_SMD:SW_Push_1P1T_NO_E-Switch_TL3301NxxxxxG, symbol Switch:SW_Push
- added SW18: Button16, Button_Switch_SMD:SW_Push_1P1T_NO_E-Switch_TL3301NxxxxxG, symbol Switch:SW_Push
- added SW19: Button17, Button_Switch_SMD:SW_Push_1P1T_NO_E-Switch_TL3301NxxxxxG, symbol Switch:SW_Push
- added SW2: BOOT, Button_Switch_SMD:SW_Push_1P1T_NO_E-Switch_TL3301NxxxxxG, symbol Switch:SW_Push
- added SW20: Button18, Button_Switch_SMD:SW_Push_1P1T_NO_E-Switch_TL3301NxxxxxG, symbol Switch:SW_Push
- added SW21: Button19, Button_Switch_SMD:SW_Push_1P1T_NO_E-Switch_TL3301NxxxxxG, symbol Switch:SW_Push
- added SW22: Button20, Button_Switch_SMD:SW_Push_1P1T_NO_E-Switch_TL3301NxxxxxG, symbol Switch:SW_Push
- added SW23: Button21, Button_Switch_SMD:SW_Push_1P1T_NO_E-Switch_TL3301NxxxxxG, symbol Switch:SW_Push
- added SW24: Button22, Button_Switch_SMD:SW_Push_1P1T_NO_E-Switch_TL3301NxxxxxG, symbol Switch:SW_Push
- added SW25: Button23, Button_Switch_SMD:SW_Push_1P1T_NO_E-Switch_TL3301NxxxxxG, symbol Switch:SW_Push
- added SW26: Button24, Button_Switch_SMD:SW_Push_1P1T_NO_E-Switch_TL3301NxxxxxG, symbol Switch:SW_Push
- added SW27: Button25, Button_Switch_SMD:SW_Push_1P1T_NO_E-Switch_TL3301NxxxxxG, symbol Switch:SW_Push
- added SW28: Button26, Button_Switch_SMD:SW_Push_1P1T_NO_E-Switch_TL3301NxxxxxG, symbol Switch:SW_Push
- added SW29: Button27, Button_Switch_SMD:SW_Push_1P1T_NO_E-Switch_TL3301NxxxxxG, symbol Switch:SW_Push
- added SW3: Button1, Button_Switch_SMD:SW_Push_1P1T_NO_E-Switch_TL3301NxxxxxG, symbol Switch:SW_Push
- added SW30: Button28, Button_Switch_SMD:SW_Push_1P1T_NO_E-Switch_TL3301NxxxxxG, symbol Switch:SW_Push
- added SW31: Button29, Button_Switch_SMD:SW_Push_1P1T_NO_E-Switch_TL3301NxxxxxG, symbol Switch:SW_Push
- added SW32: Button30, Button_Switch_SMD:SW_Push_1P1T_NO_E-Switch_TL3301NxxxxxG, symbol Switch:SW_Push
- added SW33: Button31, Button_Switch_SMD:SW_Push_1P1T_NO_E-Switch_TL3301NxxxxxG, symbol Switch:SW_Push
- added SW34: Button32, Button_Switch_SMD:SW_Push_1P1T_NO_E-Switch_TL3301NxxxxxG, symbol Switch:SW_Push
- added SW35: Button33, Button_Switch_SMD:SW_Push_1P1T_NO_E-Switch_TL3301NxxxxxG, symbol Switch:SW_Push
- added SW36: Button34, Button_Switch_SMD:SW_Push_1P1T_NO_E-Switch_TL3301NxxxxxG, symbol Switch:SW_Push
- added SW37: Button35, Button_Switch_SMD:SW_Push_1P1T_NO_E-Switch_TL3301NxxxxxG, symbol Switch:SW_Push
- added SW38: Button36, Button_Switch_SMD:SW_Push_1P1T_NO_E-Switch_TL3301NxxxxxG, symbol Switch:SW_Push
- added SW39: Button37, Button_Switch_SMD:SW_Push_1P1T_NO_E-Switch_TL3301NxxxxxG, symbol Switch:SW_Push
- added SW4: Button2, Button_Switch_SMD:SW_Push_1P1T_NO_E-Switch_TL3301NxxxxxG, symbol Switch:SW_Push
- added SW40: Button38, Button_Switch_SMD:SW_Push_1P1T_NO_E-Switch_TL3301NxxxxxG, symbol Switch:SW_Push
- added SW41: Button39, Button_Switch_SMD:SW_Push_1P1T_NO_E-Switch_TL3301NxxxxxG, symbol Switch:SW_Push
- added SW42: Button40, Button_Switch_SMD:SW_Push_1P1T_NO_E-Switch_TL3301NxxxxxG, symbol Switch:SW_Push
- added SW43: Button41, Button_Switch_SMD:SW_Push_1P1T_NO_E-Switch_TL3301NxxxxxG, symbol Switch:SW_Push
- added SW44: Button42, Button_Switch_SMD:SW_Push_1P1T_NO_E-Switch_TL3301NxxxxxG, symbol Switch:SW_Push
- added SW45: Button43, Button_Switch_SMD:SW_Push_1P1T_NO_E-Switch_TL3301NxxxxxG, symbol Switch:SW_Push
- added SW46: Button44, Button_Switch_SMD:SW_Push_1P1T_NO_E-Switch_TL3301NxxxxxG, symbol Switch:SW_Push
- added SW47: Button45, Button_Switch_SMD:SW_Push_1P1T_NO_E-Switch_TL3301NxxxxxG, symbol Switch:SW_Push
- added SW48: Button46, Button_Switch_SMD:SW_Push_1P1T_NO_E-Switch_TL3301NxxxxxG, symbol Switch:SW_Push
- added SW49: Button47, Button_Switch_SMD:SW_Push_1P1T_NO_E-Switch_TL3301NxxxxxG, symbol Switch:SW_Push
- added SW5: Button3, Button_Switch_SMD:SW_Push_1P1T_NO_E-Switch_TL3301NxxxxxG, symbol Switch:SW_Push
- added SW50: Button48, Button_Switch_SMD:SW_Push_1P1T_NO_E-Switch_TL3301NxxxxxG, symbol Switch:SW_Push
- added SW51: Button49, Button_Switch_SMD:SW_Push_1P1T_NO_E-Switch_TL3301NxxxxxG, symbol Switch:SW_Push
- added SW52: Button50, Button_Switch_SMD:SW_Push_1P1T_NO_E-Switch_TL3301NxxxxxG, symbol Switch:SW_Push
- added SW53: SW_SPDT, Button_Switch_SMD:SW_SPDT_CK_JS102011SAQN, symbol Switch:SW_SPDT
- added SW6: Button4, Button_Switch_SMD:SW_Push_1P1T_NO_E-Switch_TL3301NxxxxxG, symbol Switch:SW_Push
- added SW7: Button5, Button_Switch_SMD:SW_Push_1P1T_NO_E-Switch_TL3301NxxxxxG, symbol Switch:SW_Push
- added SW8: Button6, Button_Switch_SMD:SW_Push_1P1T_NO_E-Switch_TL3301NxxxxxG, symbol Switch:SW_Push
- added SW9: Button7, Button_Switch_SMD:SW_Push_1P1T_NO_E-Switch_TL3301NxxxxxG, symbol Switch:SW_Push
- added TP1, TP2, TP3, TP4, TP5: TestPoint, TestPoint:TestPoint_Pad_D2.0mm, symbol Connector:TestPoint
- added TP6: VBAT, TestPoint:TestPoint_THTPad_3.0x3.0mm_Drill1.5mm, symbol Connector:TestPoint
- added TP7: GND, TestPoint:TestPoint_THTPad_3.0x3.0mm_Drill1.5mm, symbol Connector:TestPoint
- added U1: ESP32-S3-WROOM-1-N16R8, opencalc_footprint_library:ESP32-S3-WROOM-1, symbol opencalc_library:ESP32-S3-WROOM-1-N16R8
- added U2: TPS63802DLAR, opencalc_footprint_library:TPS63802DLAR, symbol opencalc_library:TPS63802DLAR
- added U3: TPD2E2U06DCKR, opencalc_footprint_library:TPD2E2U06DCKR, symbol opencalc_library:TPD2E2U06DCKR
- added U4: BQ24074RGTR, opencalc_footprint_library:BQ24074RGTR, symbol opencalc_library:BQ24074RGTR
- added U5: PAM8302AADCR, opencalc_footprint_library:PAM8302AADCR, symbol opencalc_library:PAM8302AADCR
- added U6: CMS-151504-SMT-TR, opencalc_footprint_library:CMS-151504-SMT-TR, symbol opencalc_library:CMS-151504-SMT-TR
Connections:
- new net: D12.2 (A), SW11.2
- new net: C10.1, C11.2
- new net: D17.2 (A), SW16.2
- new net: J1.5, R4.2
- new net: D50.2 (A), SW49.2
- new net: J1.8, R7.2
- new net: D43.2 (A), SW42.2
- new net: D6.2 (A), SW5.2
- new net: D1.2 (A), R1.2
- new net: D23.2 (A), SW22.2
- new net: J3.11, R10.2
- new net: D8.2 (A), SW7.2
- new net: D36.2 (A), SW35.2
- new net: D52.2 (A), SW51.2
- new net: D42.2 (A), SW41.2
- new net: D5.2 (A), SW4.2
- new net: J1.6, R5.2
- new net: J1.7, R6.2
- new net: D2.1 (K), R12.1
- new net: J3.3, R9.2
- new net: D14.2 (A), SW13.2
- new net: D53.2 (A), SW52.2
- new net: D37.2 (A), SW36.2
- new net: D51.2 (A), SW50.2
- new net: L1.1, U2.7 (L2)
- new net: L1.2, U2.9 (L1)
- new net: D16.2 (A), SW15.2
- new net: D13.2 (A), SW12.2
- new net: D20.2 (A), SW19.2
- new net: D34.2 (A), SW33.2
- new net: R12.2, U4.7 (*PGOOD)
- new net: D47.2 (A), SW46.2
- new net: D19.2 (A), SW18.2
- new net: D48.2 (A), SW47.2
- new net: D26.2 (A), SW25.2
- new net: D46.2 (A), SW45.2
- new net: D32.2 (A), SW31.2
- new net: D15.2 (A), SW14.2
- new net: D39.2 (A), SW38.2
- new net: R11.2, U4.1 (TS)
- new net: R15.1, U4.12 (ILIM)
- new net: R17.1, U4.14 (TMR)
- new net: R16.2, U4.15 (ITERM)
- new net: R14.2, U4.16 (ISET)
- new net: R13.2, U4.9 (*CHG)
- new net: D25.2 (A), SW24.2
- new net: SW53.2 (B), U2.1 (EN)
- new net: D9.2 (A), SW8.2
- new net: D45.2 (A), SW44.2
- new net: D33.2 (A), SW32.2
- new net: D44.2 (A), SW43.2
- new net: R20.2, R21.1, U2.4 (FB)
- new net: D35.2 (A), SW34.2
- new net: D24.2 (A), SW23.2
- new net: D4.2 (A), SW3.2
- new net: D3.1 (K), R13.1
- new net: D7.2 (A), SW6.2
- new net: D10.2 (A), SW9.2
- new net: D31.2 (A), SW30.2
- new net: Q1.1 (G), R32.2, R8.2
- new net: D18.2 (A), SW17.2
- new net: D29.2 (A), SW28.2
- new net: C17.2, U5.4
- new net: C16.2, U5.3
- new net: D49.2 (A), SW48.2
- new net: D21.2 (A), SW20.2
- new net: D41.2 (A), SW40.2
- new net: Q1.3 (D), R33.1
- new net: D30.2 (A), SW29.2
- new net: D11.2 (A), SW10.2
- new net: D28.2 (A), SW27.2
- new net: D40.2 (A), SW39.2
- new net: D27.2 (A), SW26.2
- new net: D38.2 (A), SW37.2
- new net: D22.2 (A), SW21.2
- new net +3V3: C1.1, C14.1, C15.2, C2.1, C3.1, C4.1, C5.1, C6.1, C8.2, D2.2 (A), D3.2 (A), J1.10, Q1.2 (S), R20.1, R22.2, R23.2, R24.2, R25.2, R26.2, R27.2, R28.2, R29.2, R30.2, R31.2, R34.1, R8.1, TP1.1, U1.2 (3V3), U2.6 (VOUT), U4.5 (EN2), U5.6
- new net AMP_OUT+: U5.5, U6.P
- new net AMP_OUT-: U5.8, U6.N
- new net AUDIO_OUT: C16.1, U1.34 (IO41)
- new net AUDIO_SD: R34.2, U1.21 (IO13), U5.1
- new net BOOT_PIN: R3.1, SW2.1, TP5.1, U1.27 (IO0)
- new net COL0: D14.1 (K), D19.1 (K), D24.1 (K), D29.1 (K), D34.1 (K), D39.1 (K), D4.1 (K), D44.1 (K), D49.1 (K), D9.1 (K), U1.10 (IO17)
- new net COL1: D10.1 (K), D15.1 (K), D20.1 (K), D25.1 (K), D30.1 (K), D35.1 (K), D40.1 (K), D45.1 (K), D5.1 (K), D50.1 (K), U1.11 (IO18)
- new net COL2: D11.1 (K), D16.1 (K), D21.1 (K), D26.1 (K), D31.1 (K), D36.1 (K), D41.1 (K), D46.1 (K), D51.1 (K), D6.1 (K), U1.31 (IO38)
- new net COL3: D12.1 (K), D17.1 (K), D22.1 (K), D27.1 (K), D32.1 (K), D37.1 (K), D42.1 (K), D47.1 (K), D52.1 (K), D7.1 (K), U1.32 (IO39)
- new net COL4: D13.1 (K), D18.1 (K), D23.1 (K), D28.1 (K), D33.1 (K), D38.1 (K), D43.1 (K), D48.1 (K), D53.1 (K), D8.1 (K), U1.33 (IO40)
- new net GND: C1.2, C11.1, C12.2, C13.1, C14.2, C15.1, C17.1, C2.2, C3.2, C4.2, C5.2, C6.2, C7.1, C8.1, C9.2, D1.1 (K), J1.11, J1.12, J1.18, J3.1, J3.16, J3.17, J3.18, J3.19, J3.20, J3.8, J3.9, R10.1, R11.1, R14.1, R15.2, R16.1, R17.2, R19.1, R2.1, R21.2, R3.2, R4.1, R5.1, R6.1, R7.1, R9.1, SW1.2, SW2.2, SW53.1 (A), TP7.1, U1.1 (GND), U1.40 (GND), U1.41 (GND), U1.42 (GND), U1.43 (GND), U1.44 (GND), U1.45 (GND), U1.46 (GND), U1.47 (GND), U1.48 (GND), U1.49 (GND), U2.2 (MODE), U2.3 (AGND), U2.8 (GND), U3.3 (GND), U4.17 (EPAD), U4.4 (*CE), U4.6 (EN1), U4.8 (VSS), U5.7
- new net LCD_BACKL: J1.9, R33.2
- new net LCD_BACKL_PIN: R32.1, U1.24 (IO47)
- new net LCD_CS: J1.14, U1.18 (IO10)
- new net LCD_DC: J1.15, U1.22 (IO14)
- new net LCD_MOSI: J1.13, U1.19 (IO11)
- new net LCD_RST: J1.17, U1.8 (IO15)
- new net LCD_SCLK: J1.16, U1.20 (IO12)
- new net PWR_LED: R1.1, U1.23 (IO21)
- new net RESET_PIN: C7.2, R2.2, SW1.1, TP4.1, U1.3 (EN)
- new net ROW0: R31.1, SW3.1, SW4.1, SW5.1, SW6.1, SW7.1, U1.39 (IO1)
- new net ROW1: R30.1, SW10.1, SW11.1, SW12.1, SW8.1, SW9.1, U1.38 (IO2)
- new net ROW2: R29.1, SW13.1, SW14.1, SW15.1, SW16.1, SW17.1, U1.35 (IO42)
- new net ROW3: R28.1, SW18.1, SW19.1, SW20.1, SW21.1, SW22.1, U1.4 (IO4)
- new net ROW4: R27.1, SW23.1, SW24.1, SW25.1, SW26.1, SW27.1, U1.5 (IO5)
- new net ROW5: R26.1, SW28.1, SW29.1, SW30.1, SW31.1, SW32.1, U1.6 (IO6)
- new net ROW6: R25.1, SW33.1, SW34.1, SW35.1, SW36.1, SW37.1, U1.25 (IO48)
- new net ROW7: R24.1, SW38.1, SW39.1, SW40.1, SW41.1, SW42.1, U1.12 (IO8)
- new net ROW8: R23.1, SW43.1, SW44.1, SW45.1, SW46.1, SW47.1, U1.17 (IO9)
- new net ROW9: R22.1, SW48.1, SW49.1, SW50.1, SW51.1, SW52.1, U1.9 (IO16)
- new net USB_D+: J3.12, J3.4, U1.14 (IO20), U3.2 (IO2)
- new net USB_D-: J3.13, J3.5, U1.13 (IO19), U3.1 (IO1)
- new net USB_VBUS: C10.2, F1.2, TP3.1, U4.13 (IN)
- new net VBAT: C9.1, R18.1, TP2.1, TP6.1, U4.2 (BAT), U4.3 (BAT)
- new net VBAT_DIV: C12.1, R18.2, R19.2, U1.7 (IO7)
- new net VBUS_FUSE: F1.1, J3.10, J3.15, J3.2, J3.7
- new net VSYS: C13.2, SW53.3 (C), U2.10 (VIN), U4.10 (OUT), U4.11 (OUT)
- no-connect marks 0 -> 16
Other:
- title: (none) -> OPENCALC

Commit message: big software, readme, and blog
Parts:
- added C18, C19: 100nF, Capacitor_SMD:C_0805_2012Metric_Pad1.18x1.45mm_HandSolder, symbol Device:C
- added J2: PPTC152LFBN-RC, opencalc_footprint_library:PPTC152LFBN_RC, symbol opencalc_library:PPTC152LFBN-RC
- added R35, R36, R37: 10kΩ, Resistor_SMD:R_0805_2012Metric_Pad1.20x1.40mm_HandSolder, symbol Device:R
- added R38, R39: 4.7kΩ, Resistor_SMD:R_0805_2012Metric_Pad1.20x1.40mm_HandSolder, symbol Device:R
- added U7: ADS1115IDGST, opencalc_footprint_library:ADS1115IDGST, symbol opencalc_library:ADS1115IDGST
- added U8: MCP23017T-E/SO, opencalc_footprint_library:MCP23017T_E_SO, symbol opencalc_library:MCP23017T-E_SO
- C1, C10, C11, C12, C13, C14, C15, C16, C17, C2, C3, C4, C5, C6, C7, C8, C9: footprint Capacitor_SMD:C_0603_1608Metric -> Capacitor_SMD:C_0805_2012Metric_Pad1.18x1.45mm_HandSolder
- D1, D2, D3: footprint LED_SMD:LED_0603_1608Metric -> LED_SMD:LED_0805_2012Metric_Pad1.15x1.40mm_HandSolder
- D10, D11, D12, D13, D14, D15, D16, D17, D18, D19, D20, D21, D22, D23, D24, D25, D26, D27, D28, D29, D30, D31, D32, D33, D34, D35, D36, D37, D38, D39, D4, D40, D41, D42, D43, D44, D45, D46, D47, D48, D49, D5, D50, D51, D52, D53, D6, D7, D8, D9: footprint Diode_SMD:D_SOD-523 -> Diode_SMD:D_0805_2012Metric_Pad1.15x1.40mm_HandSolder
- R1, R10, R11, R12, R13, R14, R15, R17, R18, R19, R2, R20, R21, R22, R23, R24, R25, R26, R27, R28, R29, R3, R30, R31, R32, R33, R34, R4, R5, R6, R7, R8, R9: footprint Resistor_SMD:R_0603_1608Metric -> Resistor_SMD:R_0805_2012Metric_Pad1.20x1.40mm_HandSolder
- R16: value 4.4kΩ -> 2kΩ; footprint Resistor_SMD:R_0603_1608Metric -> Resistor_SMD:R_0805_2012Metric_Pad1.20x1.40mm_HandSolder
Connections:
- net +3V3: now also R2.1, R3.2, C18.2, C19.2, J2.1, J2.15, R35.2, R37.2, R38.2, R39.2, U7.8 (VDD), U8.9 (VDD)
- net AUDIO_SD: now also R36.2, U8.21 (GPA0); no longer U1.21 (IO13)
- net GND: now also C18.1, C19.1, J2.16, J2.18, J2.2, J2.20, J2.22, J2.24, J2.28, R36.1, U7.1 (ADDR), U7.3 (GND), U8.10 (VSS), U8.15 (A0), U8.16 (A1), U8.17 (A2); no longer R2.1, R3.2
- net PWR_LED: now also U8.22 (GPA1); no longer U1.23 (IO21)
- new net: R35.1, U8.18 (*RESET)
- new net ADS_RDY: J2.27, R37.1, U7.2 (ALERT_RDY)
- new net APIN0: J2.17, U7.4 (AIN0)
- new net APIN1: J2.19, U7.5 (AIN1)
- new net APIN2: J2.21, U7.6 (AIN2)
- new net APIN3: J2.23, U7.7 (AIN3)
- new net DPIN0: J2.3, U8.23 (GPA2)
- new net DPIN1: J2.4, U8.24 (GPA3)
- new net DPIN10: J2.13, U8.6 (GPB5)
- new net DPIN11: J2.14, U8.7 (GPB6)
- new net DPIN2: J2.5, U8.25 (GPA4)
- new net DPIN3: J2.6, U8.26 (GPA5)
- new net DPIN4: J2.7, U8.27 (GPA6)
- new net DPIN5: J2.8, U8.1 (GPB0)
- new net DPIN6: J2.9, U8.2 (GPB1)
- new net DPIN7: J2.10, U8.3 (GPB2)
- new net DPIN8: J2.11, U8.4 (GPB3)
- new net DPIN9: J2.12, U8.5 (GPB4)
- new net MCP_INTA: J2.29, U8.20 (INTA)
- new net MCP_INTB: J2.30, U8.19 (INTB)
- new net SCL: J2.26, R38.1, U1.23 (IO21), U7.10 (SCL), U8.12 (SCL)
- new net SDA: J2.25, R39.1, U1.21 (IO13), U7.9 (SDA), U8.13 (SDA)
- no-connect marks 16 -> 20

Commit message: removed files
Parts:
- R34: value 10k -> DNP; now not fitted
- R36: value 10kΩ -> 100kΩ
Connections:
- net GND: now also C10.1
- net USB_VBUS: now also C11.2
Other:
- moved on the sheet: C10
Changed lines of the file:
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@@
 	(wire
 		(pts
+			(xy 551.18 125.73) (xy 553.72 125.73)
+		)
+		(stroke
+			(width 0)
+			(type default)
+		)
+	)
+	(wire
+		(pts
+			(xy 553.72 125.73) (xy 553.72 133.35)
+		)
+		(stroke
+			(width 0)
+			(type default)
+		)
+	)
+	(wire
+		(pts
+			(xy 553.72 133.35) (xy 561.34 133.35)
+		)
+		(stroke
+			(width 0)
+			(type default)
+		)
+	)
+	(wire
+		(pts
+			(xy 551.18 118.11) (xy 561.34 118.11)
+		)
+		(stroke
+			(width 0)
+			(type default)
+		)
+	)
+	(wire
+		(pts
+			(xy 561.34 118.11) (xy 561.34 125.73)
+		)
+		(stroke
+			(width 0)
+			(type default)
+		)
+	)
+	(wire
+		(pts
 			(xy 88.9 327.66) (xy 116.84 327.66)
 		)
@@
 	(symbol
 		(lib_id "Device:C")
-		(at 551.18 129.54 0)
+		(at 561.34 129.54 0)
 		(unit 1)
 		(exclude_from_sim no)
@@
 		(fields_autoplaced yes)
 		(property "Reference" "C10"
-			(at 554.99 128.2699 0)
+			(at 565.15 128.2699 0)
 			(effects
 				(font
@@
 		)
 		(property "Value" "100nF"
-			(at 554.99 130.8099 0)
+			(at 565.15 130.8099 0)
 			(effects
 				(font
@@
 		)
 		(property "Footprint" "Capacitor_SMD:C_0805_2012Metric_Pad1.18x1.45mm_HandSolder"
-			(at 552.1452 133.35 0)
+			(at 562.3052 133.35 0)
 			(effects
 				(font
@@
 		)
 		(property "Datasheet" "~"
-			(at 551.18 129.54 0)
+			(at 561.34 129.54 0)
 			(effects
 				(font
@@
 		)
 		(property "Description" "Unpolarized capacitor"
-			(at 551.18 129.54 0)
+			(at 561.34 129.54 0)
 			(effects
 				(font
@@
 			)
 		)
-		(property "Value" "10kΩ"
+		(property "Value" "100kΩ"
 			(at 341.63 295.9099 0)
 			(effects
@@
 		(in_bom yes)
 		(on_board yes)
-		(dnp no)
+		(dnp yes)
 		(fields_autoplaced yes)
 		(property "Reference" "R34"
@@
 			)
 		)
-		(property "Value" "10k"
+		(property "Value" "DNP"
 			(at 265.43 175.2599 0)
 			(effects

Commit message: website added
Parts:
- added C20, C21: 10nF, Capacitor_SMD:C_0805_2012Metric_Pad1.18x1.45mm_HandSolder, symbol Device:C
- added R40, R41: 1kΩ, Resistor_SMD:R_0805_2012Metric_Pad1.20x1.40mm_HandSolder, symbol Device:R
- R33: value 33Ω -> 1Ω
Connections:
- net AUDIO_OUT: now also R40.1; no longer C16.1
- net GND: now also C20.2, C21.2
- new net: C16.1, C20.1, R41.2
- new net: C21.1, R40.2, R41.1
